File: VX-Line/hardware/KiCad/VX-Line_2021__original/VX-Line_original_1Layer_THT.kicad_sch (KiCad schematic)
At the start: 71 parts, among them J1 IN +, J2 IN 0 (GND), J3 IN -, J4 +UB, J5 Out, J6 Out 0 (GND), J7 UB 0 (GND), J8 -UB, Q1 2SC2240, Q2 2SA970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

Commit message: Add files via upload
Parts:
- C13, C16: value (none) -> 3x 1000µF/50V; footprint (none) -> analoghifi:CP_Radial_Black_D13.0mm_H26.0mm_P5.00mm_minimal_silk
- C14, C15, C17, C18: value (none) -> 1000µF/50V; footprint (none) -> analoghifi:CP_Radial_Black_D13.0mm_H26.0mm_P5.00mm_minimal_silk
Changed lines of the file:
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@@
       (effects (font (size 1.27 1.27)) (justify left))
     )
-    (property "Value" "" (id 1) (at 208.28 118.11 0)
-      (effects (font (size 1.27 1.27)) (justify left) hide)
-    )
-    (property "Footprint" "" (id 2) (at 210.5152 113.03 0)
+    (property "Value" "1000µF/50V" (id 1) (at 208.28 118.11 0)
+      (effects (font (size 1.27 1.27)) (justify left) hide)
+    )
+    (property "Footprint" "analoghifi:CP_Radial_Black_D13.0mm_H26.0mm_P5.00mm_minimal_silk" (id 2) (at 210.5152 113.03 0)
       (effects (font (size 1.27 1.27)) hide)
     )
@@
       (effects (font (size 1.27 1.27)) (justify left))
     )
-    (property "Value" "" (id 1) (at 194.31 118.11 0)
-      (effects (font (size 1.27 1.27)) (justify left))
-    )
-    (property "Footprint" "" (id 2) (at 197.8152 113.03 0)
+    (property "Value" "3x 1000µF/50V" (id 1) (at 194.31 118.11 0)
+      (effects (font (size 1.27 1.27)) (justify left))
+    )
+    (property "Footprint" "analoghifi:CP_Radial_Black_D13.0mm_H26.0mm_P5.00mm_minimal_silk" (id 2) (at 197.8152 113.03 0)
       (effects (font (size 1.27 1.27)) hide)
     )
@@
       (effects (font (size 1.27 1.27)) (justify left))
     )
-    (property "Value" "" (id 1) (at 205.74 15.24 0)
-      (effects (font (size 1.27 1.27)) (justify left) hide)
-    )
-    (property "Footprint" "" (id 2) (at 210.5152 34.29 0)
+    (property "Value" "1000µF/50V" (id 1) (at 205.74 15.24 0)
+      (effects (font (size 1.27 1.27)) (justify left) hide)
+    )
+    (property "Footprint" "analoghifi:CP_Radial_Black_D13.0mm_H26.0mm_P5.00mm_minimal_silk" (id 2) (at 210.5152 34.29 0)
       (effects (font (size 1.27 1.27)) hide)
     )
@@
       (effects (font (size 1.27 1.27)) (justify left))
     )
-    (property "Value" "" (id 1) (at 199.39 120.65 0)
-      (effects (font (size 1.27 1.27)) (justify left) hide)
-    )
-    (property "Footprint" "" (id 2) (at 204.1652 113.03 0)
+    (property "Value" "1000µF/50V" (id 1) (at 199.39 120.65 0)
+      (effects (font (size 1.27 1.27)) (justify left) hide)
+    )
+    (property "Footprint" "analoghifi:CP_Radial_Black_D13.0mm_H26.0mm_P5.00mm_minimal_silk" (id 2) (at 204.1652 113.03 0)
       (effects (font (size 1.27 1.27)) hide)
     )
@@
       (effects (font (size 1.27 1.27)) (justify left))
     )
-    (property "Value" "" (id 1) (at 199.39 16.51 0)
-      (effects (font (size 1.27 1.27)) (justify left) hide)
-    )
-    (property "Footprint" "" (id 2) (at 204.1652 34.29 0)
+    (property "Value" "1000µF/50V" (id 1) (at 199.39 16.51 0)
+      (effects (font (size 1.27 1.27)) (justify left) hide)
+    )
+    (property "Footprint" "analoghifi:CP_Radial_Black_D13.0mm_H26.0mm_P5.00mm_minimal_silk" (id 2) (at 204.1652 34.29 0)
       (effects (font (size 1.27 1.27)) hide)
     )
@@
       (effects (font (size 1.27 1.27)) (justify left))
     )
-    (property "Value" "" (id 1) (at 198.12 22.86 0)
-      (effects (font (size 1.27 1.27)) (justify left))
-    )
-    (property "Footprint" "" (id 2) (at 197.8152 34.29 0)
-      (effects (font (size 1.27 1.27)) hide)
-    )
+    (property "Value" "3x 1000µF/50V" (id 1) (at 198.12 22.86 0)
+      (effects (font (size 1.27 1.27)) (justify left))
+    )
+    (property "Footprint" "analoghifi:CP_Radial_Black_D13.0mm_H26.0mm_P5.00mm_minimal_silk" (id 2) (at 197.8152 34.29 0)
+      (effects (font (size 1.27 1.27)) hide)
+    )
